File: speeduino_48p/Fuel_Ignition.kicad_sch (KiCad schematic)
At the start: 49 parts, among them U1 VNLD5090, U2 IXDN602, U3 VNLD5090, U4 IXDN602

Commit message: v1.1
Other:
- title: Speeduino XM -> Speeduino 48p
Changed lines of the file:
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@@
 	(paper "A4")
 	(title_block
-		(title "Speeduino XM")
-		(date "2026-01-11")
-		(rev "1.0")
+		(title "Speeduino 48p")
+		(date "2026-02-07")
+		(rev "1.1")
 		(company "Louis")
 	)
