File: speeduino_48p/connector.kicad_sch (KiCad schematic)
At the start: 5 parts, among them J10 Delphi_Sicma_24, J2 Conn_01x06, J9 Delphi_Sicma_24

Commit message: v1.1
Parts:
- added J1: Conn_01x02, Connector_PinHeader_2.54mm:PinHeader_1x02_P2.54mm_Vertical, symbol Connector_Generic:Conn_01x02
Connections:
- net FAN-OUT: now also J9.C5; no longer J9.C6
- net FUELPUMP-OUT: now also J9.C6; no longer J9.C7
- net GND: now also J10.C8, J9.C8; no longer J10.B5, J10.B6, J10.C2, J10.C3, J9.C5
- net MAP-EXT: now also J10.B6; no longer J10.C8
- net TACHO-OUT: now also J9.C7; no longer J9.C8
- net VDDA: now also J10.C2, J10.C3; no longer J10.B3, J10.B4
- new net MCU-D14: J1.2 (Pin_2), J10.B4
- new net MCU-D15: J1.1 (Pin_1), J10.B3
- no-connect marks 0 -> 1
Other:
- note added: "RX"
- note added: "SERIAL3"
- note added: "TX"
- title: Speeduino XM -> Speeduino 48p
