File: speeduino_48p/inputs.kicad_sch (KiCad schematic)
At the start: 44 parts, among them IC3 Trig Cond Socket, U5 MPXA4250, U6 SP720

Commit message: v1.1
Parts:
- added R58: 51k, Resistor_SMD:R_0805_2012Metric, symbol Device:R
- C1: value 0.01uF -> 0.1uF
- C29, C8: value 470pf -> 47pf
- U5: value MPXA4250 -> MPXHxxxx; footprint Package_SO:SOP-8_6.605x9.655mm_P2.54mm -> Package_SO:SOP-8_3.76x4.96mm_P1.27mm; Digikey Part Number MPX4250AP-ND -> MPXH6400A; Manufacturer_Part_Number MPX4250AP -> MPXH6400A; URL https://www.digikey.com.au/product-detail/en/nxp-usa-inc/MP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 -> (none)
Connections:
- net ADC-Clamp-2: no longer C8.2
- net GND: now also R58.1
- net MAP-EXT: now also C8.2
- net at JP11.2 (C), U5.4 (VOUT): now also R58.2
Other:
- note added: "MPXH6400A - 4bar MPXHZ6250AC6T1 - 2.5bar"
- title: Speeduino XM -> Speeduino 48p
- moved on the sheet: C1, C2, C8, R34, U5
