File: speeduino_48p/outputs.kicad_sch (KiCad schematic)
At the start: 19 parts, among them Q1 SSM3K357R, Q2 SSM3K357R, Q3 SSM3K357R, U7 VNLD5090, U9 VNLD5090

Commit message: v1.1
Other:
- title: Speeduino XM -> Speeduino 48p
Changed lines of the file:
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@@
 	(paper "A4")
 	(title_block
-		(title "Speeduino XM")
-		(date "2026-01-11")
-		(rev "1.0")
+		(title "Speeduino 48p")
+		(date "2026-02-07")
+		(rev "1.1")
 		(company "Louis")
 	)
