File: speeduino_48p/proto.kicad_sch (KiCad schematic)
At the start: 7 parts, among them J5 Conn_01x04

Commit message: v1.1
Other:
- title: Speeduino XM -> Speeduino 48p
Changed lines of the file:
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@@
 	(paper "A4")
 	(title_block
-		(title "Speeduino XM")
-		(date "2026-01-11")
-		(rev "1.0")
+		(title "Speeduino 48p")
+		(date "2026-02-07")
+		(rev "1.1")
 		(company "Louis")
 	)
