File: speeduino_48p/speeduino_48p.kicad_pcb (KiCad board)
At the start: 2 copper layers, 116.5 x 98 mm, 141 parts, among them IC3 Trig Cond Socket, J10 Delphi_Sicma_24, J2 Conn_01x06, J5 Conn_01x04, J9 Delphi_Sicma_24, Q1 SSM3K357R, Q2 SSM3K357R, Q3 SSM3K357R, U1 VNLD5090, U10 MEGA_PRO_EMBED_CH340G___ATMEG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, U2 IXDN602, U3 VNLD5090, U4 IXDN602, U5 MPXA4250, U6 SP720, U7 VNLD5090, U8 LM2940S-5.0/NOPB, U9 VNLD5090

Commit message: v1.1
Parts:
- added G***: LOGO, LOGO, F.Cu at (173.4, 129.4)
- added G***: LOGO, LOGO, B.Cu at (121.3, 93.2)
- added J1: Conn_01x02, Connector_PinHeader_2.54mm:PinHeader_1x02_P2.54mm_Vertical, F.Cu at (184.5, 111.3)
- added R58: 51k, Resistor_SMD:R_0805_2012Metric, F.Cu at (177.4, 55.9)
- C1: value 0.01uF -> 0.1uF
- C29, C8: value 470pf -> 47pf
- H1, H2, H3, H4: renamed from ?; value (none) -> MountingHole; footprint (none) -> MountingHole:MountingHole_3.2mm_M3_DIN965_Pad
- U5: value MPXA4250 -> MPXHxxxx; footprint Package_SO:SOP-8_6.605x9.655mm_P2.54mm -> Package_SO:SOP-8_3.76x4.96mm_P1.27mm
- moved H4 10.7 mm to (198.0, 137.1)
- moved H3 6.39 mm to (114.9, 137.1)
- moved U5 6.20 mm to (180.9, 51.4)
- moved C1 4.32 mm to (173.9, 49.7)
- moved C2 4.32 mm to (176.1, 49.7)
- moved C8 3.27 mm to (173.2, 66.1), turned to 90 degrees
- moved R34 3.24 mm to (175.3, 66.1)
- moved C29 1.42 mm to (183.9, 67.0), turned to 90 degrees
Connections:
- C8 pad 2: ADC-Clamp-2 -> MAP-EXT
- J10 pad B3: VDDA -> MCU-D15
- J10 pad B4: VDDA -> MCU-D14
- J10 pad B5: GND -> unconnected-(J10-PadB5)
- J10 pad B6: GND -> MAP-EXT
- J10 pad C2: GND -> VDDA
- J10 pad C3: GND -> VDDA
- J10 pad C8: MAP-EXT -> GND
- J9 pad C5: GND -> FAN-OUT
- J9 pad C6: FAN-OUT -> FUELPUMP-OUT
- J9 pad C7: FUELPUMP-OUT -> TACHO-OUT
- J9 pad C8: TACHO-OUT -> GND
Routing:
- net MCU-D14: track 0.00 -> 111.3 mm, vias 0 -> 2
- net MCU-D15: track 0.00 -> 110.0 mm, vias 0 -> 2
- net ADC-Clamp-2: track 46.9 -> 40.9 mm
- net TACHO-OUT: track 24.3 -> 28.7 mm
- net VDD: track 278.7 -> 282.8 mm
- net MAP-EXT: track 90.7 -> 94.7 mm
- net Net-(JP11-C): track 4.55 -> 8.52 mm
- net ADC-Clamp-10: track 91.6 -> 95.5 mm
- net FUELPUMP-OUT: track 19.3 -> 22.9 mm
- net FAN-OUT: track 22.2 -> 25.6 mm
- net VDDA: track 115.2 -> 113.8 mm
- net 12V-SW: track 265.7 -> 265.2 mm
- net GND: vias 295 -> 328
Other:
- outline, holes or cut-outs redrawn
- board text added: "JLCJLCJLCJLC"
- board text added: "NC"
- board text added: "Powered by"
- board text added: "RX TX"
- board text added: "This board is based on Speeduino v0.4.4d design and aims to provide a low-cost, all in one ECU. More information : https://github.com/Blackbird128/speeduino_48pin"
- board text added: "speeduino_48pin"
- board text added: "v1.1 Louis 2026"
- board text removed: "Louis 2025 v1.0"
- board text removed: "Speeduino 48 SMD"
- board text removed: "Speeduino v0.4.4d compatible"
- board text removed: "based on speeduino 0.4.4d by Josh Stewart"
- board text removed: "based on speeduino V0.4.4d by Josh Stewart"
