File: speeduino_48p/speeduino_48p.kicad_sch (KiCad schematic)
At the start: 1 part, among them U10 MEGA_PRO_EMBED_CH340G___ATMEG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

Commit message: v1.1
Parts:
- added H1, H2, H3, H4: MountingHole, MountingHole:MountingHole_3.2mm_M3_DIN965_Pad, symbol Mechanical:MountingHole
Other:
- title: Speeduino XM -> Speeduino 48p
